Commit message: added 2D lidar and stacked into pointcloud

File: src/vehicle_simulator/urdf/lidar.urdf.xacro (robot description, xacro)
@@ -2,6 +2,10 @@
 <robot xmlns:xacro="http://www.ros.org/wiki/xacro" name="example">
   <link name="lidar" />
-  <xacro:include filename="$(find velodyne_description)/urdf/VLP-16.urdf.xacro"/>
+  <!-- <xacro:include filename="$(find velodyne_description)/urdf/VLP-16.urdf.xacro"/>
   <xacro:VLP-16 parent="lidar" name="velodyne" topic="/velodyne_points" hz="6.3" samples="350" min_range="0.1">
+    <origin xyz="0 0 0" rpy="0 0 0" />
+  </xacro:VLP-16> -->
+  <xacro:include filename="$(find velodyne_description)/urdf/lidar_2D.urdf.xacro"/>
+  <xacro:VLP-16 parent="lidar" name="rplidar" topic="/scan" hz="5" samples="350" min_range="0.1" organize_cloud="true">
     <origin xyz="0 0 0" rpy="0 0 0" />
   </xacro:VLP-16>
